File: RAK3172-Breakout.brd (EAGLE design)
At the start: 50 x 23.2 mm, 26 parts, among them J1 FTDI, J3 JTAG, SW1 RESET, SW2 BOOT0

Commit message: Bump to V1.1
Parts:
- C4, C5, C6: value 10uF -> 100uF
Connections:
- net 3V3: now also SW2.2
- net GND: no longer SW2.2
Routing:
- net 3V3: track 79.0 -> 85.9 mm
Other:
- board text added: "RAK3172 Mini V1.1"
- board text added: "V1.1"
- board text removed: "RAK3172 Mini V1.0"
- board text removed: "V1.0"
Changed lines of the file:
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@@
 <text x="11.6205" y="23.562" size="0.889" layer="25" font="vector" ratio="15" align="center">Reset</text>
 <text x="11.557" y="1.965" size="0.889" layer="25" font="vector" ratio="15" rot="R180" align="center">Boot</text>
-<text x="7.366" y="12.192" size="1.27" layer="22" font="vector" ratio="15" rot="MR270" align="center">RAK3172 Mini V1.0</text>
+<text x="7.366" y="12.192" size="1.27" layer="22" font="vector" ratio="15" rot="MR270" align="center">RAK3172 Mini V1.1</text>
 <text x="33.02" y="10.795" size="0.889" layer="37" ratio="12">U1</text>
 <text x="9.779" y="6.29" size="0.8128" layer="25" font="vector" ratio="15" rot="R180" align="center">GND</text>
@@
 <text x="3.683" y="6.417" size="0.8128" layer="26" font="vector" ratio="15" rot="MR180" align="center">GND</text>
 <text x="44.069" y="16.129" size="1.27" layer="21" font="vector" ratio="15" rot="R270" align="center">RAK3172</text>
-<text x="48.514" y="18.542" size="1.27" layer="21" font="vector" ratio="15" rot="R90" align="center">V1.0</text>
+<text x="48.514" y="18.542" size="1.27" layer="21" font="vector" ratio="15" rot="R90" align="center">V1.1</text>
 <dimension x1="0" y1="-6.35" x2="50.165" y2="-6.35" x3="25.0825" y3="-16.51" textsize="1.778" layer="47"/>
 <dimension x1="-9.525" y1="0" x2="-9.525" y2="22.86" x3="-15.875" y3="11.43" textsize="1.778" layer="47"/>
@@
 </element>
 <element name="COIN1" library="_c2h" package="CR2450-SMD" value="CR2450" x="27.559" y="12.7" smashed="yes" rot="MR0"/>
-<element name="C4" library="_c2h" package="0805-CAP" value="10uF" x="14.605" y="19.685" smashed="yes" rot="MR270"/>
-<element name="C5" library="_c2h" package="0805-CAP" value="10uF" x="12.7" y="19.685" smashed="yes" rot="MR270"/>
-<element name="C6" library="_c2h" package="0805-CAP" value="10uF" x="10.795" y="19.685" smashed="yes" rot="MR270"/>
+<element name="C4" library="_c2h" package="0805-CAP" value="100uF" x="14.605" y="19.685" smashed="yes" rot="MR270"/>
+<element name="C5" library="_c2h" package="0805-CAP" value="100uF" x="12.7" y="19.685" smashed="yes" rot="MR270"/>
+<element name="C6" library="_c2h" package="0805-CAP" value="100uF" x="10.795" y="19.685" smashed="yes" rot="MR270"/>
 <element name="C7" library="_c2h" package="0805-CAP" value="100uF" x="8.89" y="19.685" smashed="yes" rot="MR270"/>
 </elements>
@@
 <contactref element="U$3" pad="17"/>
 <contactref element="SW1" pad="1"/>
-<contactref element="SW2" pad="2"/>
 <contactref element="C2" pad="1"/>
 <contactref element="J4" pad="7"/>
@@
 <via x="42.926" y="17.78" extent="1-16" drill="0.3048"/>
 <via x="27.3685" y="6.50875" extent="1-16" drill="0.3048"/>
-<via x="12.954" y="6.604" extent="1-16" drill="0.254" diameter="0.508"/>
+<via x="10.668" y="5.334" extent="1-16" drill="0.254" diameter="0.508"/>
 <via x="33.528" y="11.176" extent="1-16" drill="0.3048"/>
 <via x="32.258" y="15.621" extent="1-16" drill="0.3048"/>
@@
 <wire x1="14.605" y1="18.685" x2="14.605" y2="18.415" width="0.4064" layer="16"/>
 <wire x1="14.605" y1="18.415" x2="15.24" y2="17.78" width="0.4064" layer="16"/>
+<contactref element="SW2" pad="2"/>
+<wire x1="9.53" y1="3.81" x2="10.668" y2="3.81" width="0.3048" layer="1"/>
+<wire x1="10.668" y1="3.81" x2="13.065" y2="6.207" width="0.3048" layer="1"/>
+<wire x1="13.065" y1="8.636" x2="13.065" y2="6.207" width="0.3048" layer="1"/>
 </signal>
 <signal name="D3">
