File: RAK3172-Breakout.sch (EAGLE design)
At the start: 24 parts, among them J1 FTDI, J3 JTAG, SW1 RESET, SW2 BOOT0

Commit message: Bump to V1.1
Parts:
- C4, C5, C6: value 10uF -> 100uF
Connections:
- net 3V3: now also SW2.2
- net GND: no longer SW2.2
Other:
- moved on the sheet: SW2
